Commit message: fixed the structure and values of Lidar and Diff_drive gazebo plugins

File: src/robocops_gazebo/description/gazebo_control.xacro (robot description, xacro)
@@ -6,6 +6,6 @@
             <left_joint>left_wheel_joint</left_joint>
             <right_joint>right_wheel_joint</right_joint>
-            <wheel_separation>0.297</wheel_separation>
-            <wheel_radius>0.033</wheel_radius>
+            <wheel_separation>0.32</wheel_separation>
+            <wheel_radius>0.06</wheel_radius>
             <!-- Limits -->
             <!-- <max_wheel_torque>200</max_wheel_torque> -->
@@ -18,4 +18,7 @@
             <odom_topic>odom</odom_topic>
             <odom_publisher_frequency>30</odom_publisher_frequency>
+            <publish_odom>true</publish_odom>
+            <publish_odom_tf>true</publish_odom_tf>
+            <publish_wheel_tf>true</publish_wheel_tf>
             <tf_topic>/tf</tf_topic>
         </plugin>

File: src/robocops_gazebo/description/lidar.xacro (robot description, xacro)
@@ -2,5 +2,5 @@
 <robot xmlns:xacro="http://www.ros.org/wiki/xacro" >
     <joint name="laser_joint" type="fixed">
-        <parent link="chassis"/>
+        <parent link="base_link"/>
         <child link="laser_frame"/>
         <origin xyz="0.122 0 0.212" rpy="0 0 0"/>
@@ -9,12 +9,6 @@
         <visual>
             <geometry>
+                <origin xyz="0 0 0" rpy="0 0 0" />
                 <cylinder radius="0.05" length="0.04"/>
-            </geometry>
-            <material name="black"/>
-        </visual>
-        <visual>
-            <origin xyz="0 0 -0.05"/>
-            <geometry>
-                <cylinder radius="0.01" length="0.1"/>
             </geometry>
             <material name="black"/>
