Commit message: change lidar rotation yaw

File: src/robocops_description/description/urdf/lidar.xacro (robot description, xacro)
@@ -4,5 +4,5 @@
         <parent link="chassis"/>
         <child link="laser_frame"/>
-        <origin xyz="0.26855 0 0.12525" rpy="0 0 0"/>
+        <origin xyz="0.26855 0 0.12525" rpy="0 0 1.5708"/>
     </joint>
     <link name="laser_frame">

Commit message: fix lidar orientation

File: src/robocops_description/description/urdf/lidar.xacro (robot description, xacro)
@@ -4,5 +4,5 @@
         <parent link="chassis"/>
         <child link="laser_frame"/>
-        <origin xyz="0.26855 0 0.12525" rpy="0 0 1.5708"/>
+        <origin xyz="0.26855 0 0.12525" rpy="0 0 -1.5708"/>
     </joint>
     <link name="laser_frame">
