Commit message: Nav2 fine tune tests 2

File: src/robocops_description/description/urdf/robot_core.xacro (robot description, xacro)
@@ -125,9 +125,9 @@
     </gazebo>
     <!-- LEFT FRONT WHEEL -->
-    <joint name="left_front_wheel_joint" type="continuous">
+    <joint name="left_front_wheel_joint" type="fixed">
         <parent link="chassis"/>
         <child link="left_front_wheel"/>
         <origin xyz="${small_wheel_offset_x} ${wheel_offset_y + small_wheel_thickness/2} ${-small_wheel_offset_z}" rpy="${-pi/2} 0 0" />
-        <axis xyz="0 0 1"/>
+        <!-- <axis xyz="0 0 1"/> -->
     </joint>
     <link name="left_front_wheel">
@@ -153,9 +153,9 @@
     </gazebo>
     <!-- RIGHT FRONT WHEEL -->
-    <joint name="right_front_wheel_joint" type="continuous">
+    <joint name="right_front_wheel_joint" type="fixed">
         <parent link="chassis"/>
         <child link="right_front_wheel"/>
         <origin xyz="${small_wheel_offset_x} ${-wheel_offset_y - small_wheel_thickness/2} ${-small_wheel_offset_z}" rpy="${pi/2} 0 0" />
-        <axis xyz="0 0 -1"/>
+        <!-- <axis xyz="0 0 -1"/> -->
     </joint>
     <link name="right_front_wheel">

Commit message: add brush fram id

File: src/robocops_description/description/urdf/robot_core.xacro (robot description, xacro)
@@ -45,4 +45,11 @@
     </joint>
     <link name="base_footprint" />
+    <!-- Burshes -->
+    <joint name="brushes_joint" type="fixed">
+        <parent link="base_link"/>
+        <child link="brushes"/>
+        <origin xyz="0.20 0 0" rpy="0 0 0"/>
+    </joint>
+    <link name="brushes" />
     <!-- CHASSIS LINK -->
     <joint name="chassis_joint" type="fixed">

Commit message: change origin of base link

File: src/robocops_description/description/urdf/robot_core.xacro (robot description, xacro)
@@ -36,13 +36,13 @@
         <color rgba="0 1 0 1"/>
     </material>
+    <link name="base_footprint" />
     <!-- BASE LINK -->
     <link name="base_link" />
     <!-- BASE_FOOTPRINT LINK -->
     <joint name="base_footprint_joint" type="fixed">
-        <parent link="base_link"/>
-        <child link="base_footprint"/>
-        <origin xyz="0 0 0" rpy="0 0 0"/>
+        <parent link="base_footprint"/>
+        <child link="base_link"/>
+        <origin xyz="-{wheel_offset_x} 0 0" rpy="0 0 0"/>
     </joint>
-    <link name="base_footprint" />
     <!-- Burshes -->
     <joint name="brushes_joint" type="fixed">
@@ -83,5 +83,5 @@
         <parent link="chassis"/>
         <child link="left_wheel"/>
-        <origin xyz="${-wheel_offset_x} ${wheel_offset_y + wheel_thickness/2} ${-wheel_offset_z}" rpy="-${pi/2} 0 0" />
+        <origin xyz="0 ${wheel_offset_y + wheel_thickness/2} ${-wheel_offset_z}" rpy="-${pi/2} 0 0" />
         <axis xyz="0 0 1"/>
     </joint>
@@ -109,5 +109,5 @@
         <parent link="chassis"/>
         <child link="right_wheel"/>
-        <origin xyz="${-wheel_offset_x} ${-wheel_offset_y - wheel_thickness/2} ${-wheel_offset_z}" rpy="${pi/2} 0 0" />
+        <origin xyz="0 ${-wheel_offset_y - wheel_thickness/2} ${-wheel_offset_z}" rpy="${pi/2} 0 0" />
         <axis xyz="0 0 -1"/>
     </joint>

Commit message: change robot desci

File: src/robocops_description/description/urdf/robot_core.xacro (robot description, xacro)
@@ -43,5 +43,5 @@
         <parent link="base_footprint"/>
         <child link="base_link"/>
-        <origin xyz="-{wheel_offset_x} 0 0" rpy="0 0 0"/>
+        <origin xyz="-${wheel_offset_x} 0 0" rpy="0 0 0"/>
     </joint>
     <!-- Burshes -->

Commit message: update urdf

File: src/robocops_description/description/urdf/robot_core.xacro (robot description, xacro)
@@ -36,18 +36,18 @@
         <color rgba="0 1 0 1"/>
     </material>
-    <link name="base_footprint" />
     <!-- BASE LINK -->
     <link name="base_link" />
     <!-- BASE_FOOTPRINT LINK -->
     <joint name="base_footprint_joint" type="fixed">
-        <parent link="base_footprint"/>
-        <child link="base_link"/>
-        <origin xyz="-${wheel_offset_x} 0 0" rpy="0 0 0"/>
+        <parent link="base_link"/>
+        <child link="base_footprint"/>
+        <origin xyz="0 0 0" rpy="0 0 0"/>
     </joint>
+    <link name="base_footprint" />
     <!-- Burshes -->
     <joint name="brushes_joint" type="fixed">
         <parent link="base_link"/>
         <child link="brushes"/>
-        <origin xyz="0.20 0 0" rpy="0 0 0"/>
+        <origin xyz="0.20 + ${wheel_offset_x}  0 0" rpy="0 0 0"/>
     </joint>
     <link name="brushes" />
@@ -56,5 +56,5 @@
         <parent link="base_link"/>
         <child link="chassis"/>
-        <origin xyz="0 0 ${chassis_height/2}"/>
+        <origin xyz="${wheel_offset_x} 0 ${chassis_height/2}"/>
     </joint>
     <link name="chassis">

Commit message: update sum

File: src/robocops_description/description/urdf/robot_core.xacro (robot description, xacro)
@@ -49,5 +49,5 @@
         <parent link="base_link"/>
         <child link="brushes"/>
-        <origin xyz="0.20 + ${wheel_offset_x}  0 0" rpy="0 0 0"/>
+        <origin xyz="${0.20 + wheel_offset_x}  0 0" rpy="0 0 0"/>
     </joint>
     <link name="brushes" />

Commit message: changfe urdf

File: src/robocops_description/description/urdf/robot_core.xacro (robot description, xacro)
@@ -81,5 +81,5 @@
     <!-- LEFT WHEEL LINK -->
     <joint name="left_wheel_joint" type="continuous">
-        <parent link="chassis"/>
+        <parent link="base_link"/>
         <child link="left_wheel"/>
         <origin xyz="0 ${wheel_offset_y + wheel_thickness/2} ${-wheel_offset_z}" rpy="-${pi/2} 0 0" />
@@ -107,5 +107,5 @@
     <!-- RIGHT WHEEL LINK -->
     <joint name="right_wheel_joint" type="continuous">
-        <parent link="chassis"/>
+        <parent link="base_link"/>
         <child link="right_wheel"/>
         <origin xyz="0 ${-wheel_offset_y - wheel_thickness/2} ${-wheel_offset_z}" rpy="${pi/2} 0 0" />

Commit message: add imu in urdf

File: src/robocops_description/description/urdf/robot_core.xacro (robot description, xacro)
@@ -45,4 +45,10 @@
     </joint>
     <link name="base_footprint" />
+    <joint name="imu_joint" type="fixed">
+        <parent link="base_link"/>
+        <child link="imu"/>
+        <origin xyz="0 0 0" rpy="0 0 0"/>
+    </joint>
+    <link name="imu" />
     <!-- Burshes -->
     <joint name="brushes_joint" type="fixed">

Commit message: update tree + imu description

File: src/robocops_description/description/urdf/robot_core.xacro (robot description, xacro)
@@ -48,5 +48,5 @@
         <parent link="base_link"/>
         <child link="imu"/>
-        <origin xyz="0 0 0" rpy="0 0 0"/>
+        <origin xyz="0 0 0" rpy="-3.14 0 -1.6"/>
     </joint>
     <link name="imu" />

Commit message: reset desc

File: src/robocops_description/description/urdf/robot_core.xacro (robot description, xacro)
@@ -48,5 +48,5 @@
         <parent link="base_link"/>
         <child link="imu"/>
-        <origin xyz="0 0 0" rpy="-3.14 0 -1.6"/>
+        <origin xyz="0 0 0" rpy="0 0 0"/>
     </joint>
     <link name="imu" />

Commit message: test door open and change urdf

File: src/robocops_description/description/urdf/robot_core.xacro (robot description, xacro)
@@ -48,5 +48,5 @@
         <parent link="base_link"/>
         <child link="imu"/>
-        <origin xyz="0 0 0" rpy="0 0 0"/>
+        <origin xyz="0 0 0" rpy="3.14 0 0"/>
     </joint>
     <link name="imu" />

Commit message: test serial with markers

File: src/robocops_description/description/urdf/robot_core.xacro (robot description, xacro)
@@ -48,5 +48,5 @@
         <parent link="base_link"/>
         <child link="imu"/>
-        <origin xyz="0 0 0" rpy="3.14 0 0"/>
+        <origin xyz="0 0 0" rpy="0 0 0"/>
     </joint>
     <link name="imu" />

Commit message: change imu position

File: src/robocops_description/description/urdf/robot_core.xacro (robot description, xacro)
@@ -48,5 +48,5 @@
         <parent link="base_link"/>
         <child link="imu"/>
-        <origin xyz="0 0 0" rpy="0 0 0"/>
+        <origin xyz="0 0 0" rpy="0 3.14 -1.57079632679"/>
     </joint>
     <link name="imu" />

Commit message: change pitch

File: src/robocops_description/description/urdf/robot_core.xacro (robot description, xacro)
@@ -48,5 +48,5 @@
         <parent link="base_link"/>
         <child link="imu"/>
-        <origin xyz="0 0 0" rpy="0 3.14 -1.57079632679"/>
+        <origin xyz="0 0 0" rpy="0 0 -1.57079632679"/>
     </joint>
     <link name="imu" />

Commit message: ciao bello

File: src/robocops_description/description/urdf/robot_core.xacro (robot description, xacro)
@@ -48,5 +48,5 @@
         <parent link="base_link"/>
         <child link="imu"/>
-        <origin xyz="0 0 0" rpy="0 0 -1.57079632679"/>
+        <origin xyz="0 0 0" rpy="0 0 0"/>
     </joint>
     <link name="imu" />

Commit message: change orientation

File: src/robocops_description/description/urdf/robot_core.xacro (robot description, xacro)
@@ -48,5 +48,5 @@
         <parent link="base_link"/>
         <child link="imu"/>
-        <origin xyz="0 0 0" rpy="0 0 0"/>
+        <origin xyz="0 0 0" rpy="0 3.14 1.57"/>
     </joint>
     <link name="imu" />

Commit message: change description

File: src/robocops_description/description/urdf/robot_core.xacro (robot description, xacro)
@@ -48,5 +48,6 @@
         <parent link="base_link"/>
         <child link="imu"/>
-        <origin xyz="0 0 0" rpy="0 3.14 1.57"/>
+        <origin xyz="0 0 0" rpy="0 0 0"/>
+        <!-- <origin xyz="0 0 0" rpy="0 3.14 1.57"/> -->
     </joint>
     <link name="imu" />

Commit message: fix imu orientation

File: src/robocops_description/description/urdf/robot_core.xacro (robot description, xacro)
@@ -48,6 +48,6 @@
         <parent link="base_link"/>
         <child link="imu"/>
-        <origin xyz="0 0 0" rpy="0 0 0"/>
-        <!-- <origin xyz="0 0 0" rpy="0 3.14 1.57"/> -->
+        <!-- <origin xyz="0 0 0" rpy="0 0 0"/> -->
+        <origin xyz="0 0 0" rpy="0 3.14 1.57"/>
     </joint>
     <link name="imu" />

Commit message: change to minus

File: src/robocops_description/description/urdf/robot_core.xacro (robot description, xacro)
@@ -49,5 +49,5 @@
         <child link="imu"/>
         <!-- <origin xyz="0 0 0" rpy="0 0 0"/> -->
-        <origin xyz="0 0 0" rpy="0 3.14 1.57"/>
+        <origin xyz="0 0 0" rpy="0 3.14 -1.57"/>
     </joint>
     <link name="imu" />

Commit message: update brushes frame

File: src/robocops_description/description/urdf/robot_core.xacro (robot description, xacro)
@@ -56,5 +56,5 @@
         <parent link="base_link"/>
         <child link="brushes"/>
-        <origin xyz="${0.20 + wheel_offset_x}  0 0" rpy="0 0 0"/>
+        <origin xyz="${0.12 + wheel_offset_x}  0 0" rpy="0 0 0"/>
     </joint>
     <link name="brushes" />

Commit message: change x offset

File: src/robocops_description/description/urdf/robot_core.xacro (robot description, xacro)
@@ -56,5 +56,5 @@
         <parent link="base_link"/>
         <child link="brushes"/>
-        <origin xyz="${0.12 + wheel_offset_x}  0 0" rpy="0 0 0"/>
+        <origin xyz="${0.05 + wheel_offset_x}  0 0" rpy="0 0 0"/>
     </joint>
     <link name="brushes" />
