Commit message: Change camera package to duplo package + add buffer + change robocops_msgs

File: src/robocops_description/description/urdf/camera.xacro (robot description, xacro)
@@ -7,5 +7,5 @@
         <origin xyz="0.0338505 0 0.00142"/>
     </joint>
-    <link name="camera">
+    <link name="camera_oak">
         <visual>
             <origin xyz="0 0 0"/>
@@ -25,6 +25,13 @@
         </xacro:inertial_box>
     </link>
-    <gazebo reference="camera">
+    <gazebo reference="camera_oak">
         <material>Gazebo/Black</material>
     </gazebo>
+    <joint name="camera_point_joint" type="fixed">
+        <parent link="camera_oak"/>
+        <child link="camera"/>
+        <origin xyz="0.05 0 0"/>
+    </joint>
+    <!-- This is the link that is centered on the rgb sensor and should be used for transform -->
+    <link name="camera"/>
 </robot>

Commit message: update camera xacro

File: src/robocops_description/description/urdf/camera.xacro (robot description, xacro)
@@ -31,5 +31,5 @@
         <parent link="camera_oak"/>
         <child link="camera"/>
-        <origin xyz="0.05 0 0"/>
+        <origin xyz="0.001 0 0.005"/>
     </joint>
     <!-- This is the link that is centered on the rgb sensor and should be used for transform -->

Commit message: fix description problem

File: src/robocops_description/description/urdf/camera.xacro (robot description, xacro)
@@ -3,5 +3,5 @@
     <joint name="camera_joint" type="fixed">
         <parent link="camera_holder2"/>
-        <child link="camera"/>
+        <child link="camera_oak"/>
         <!-- 0.025 (from axis to end) + 0.017701/2=0.0338505 -->
         <origin xyz="0.0338505 0 0.00142"/>

File: src/robocops_description/description/urdf/robot.urdf.xacro (robot description, xacro)
@@ -4,6 +4,6 @@
     <xacro:include filename="robot_core.xacro" />
     <xacro:include filename="lidar.xacro" />
-    <!-- <xacro:include filename="camera_holder.xacro" />
-    <xacro:include filename="camera.xacro" /> -->
+    <xacro:include filename="camera_holder.xacro" />
+    <xacro:include filename="camera.xacro" />
     <xacro:if value="$(arg simulation)">
         <xacro:include filename="$(find robocops_description)/description/control/gazebo_control.xacro"/>

Commit message: change camera value

File: src/robocops_description/description/urdf/camera.xacro (robot description, xacro)
@@ -1,4 +1,6 @@
 <?xml version="1.0"?>
 <robot xmlns:xacro="http://www.ros.org/wiki/xacro" >
+    <xacro:property name="tilt_deg_cam" value="25"/>
+    <xacro:property name="tilt_rad_cam" value="${tilt_deg_cam * pi / 180.0}"/>
     <joint name="camera_joint" type="fixed">
         <parent link="camera_holder2"/>
@@ -29,7 +31,7 @@
     </gazebo>
     <joint name="camera_point_joint" type="fixed">
-        <parent link="camera_oak"/>
+        <parent link="base_link"/>
         <child link="camera"/>
-        <origin xyz="0.001 0 0.005"/>
+        <origin xyz="37 0 17.65" rpy="0 ${tilt_rad_cam} 0"/>
     </joint>
     <!-- This is the link that is centered on the rgb sensor and should be used for transform -->

Commit message: change units

File: src/robocops_description/description/urdf/camera.xacro (robot description, xacro)
@@ -33,5 +33,5 @@
         <parent link="base_link"/>
         <child link="camera"/>
-        <origin xyz="37 0 17.65" rpy="0 ${tilt_rad_cam} 0"/>
+        <origin xyz="0.037 0 0.01765" rpy="0 ${tilt_rad_cam} 0"/>
     </joint>
     <!-- This is the link that is centered on the rgb sensor and should be used for transform -->

Commit message: change unit

File: src/robocops_description/description/urdf/camera.xacro (robot description, xacro)
@@ -33,5 +33,5 @@
         <parent link="base_link"/>
         <child link="camera"/>
-        <origin xyz="0.037 0 0.01765" rpy="0 ${tilt_rad_cam} 0"/>
+        <origin xyz="0.37 0 0.1765" rpy="0 ${tilt_rad_cam} 0"/>
     </joint>
     <!-- This is the link that is centered on the rgb sensor and should be used for transform -->

Commit message: fix camera angle

File: src/robocops_description/description/urdf/camera.xacro (robot description, xacro)
@@ -1,5 +1,5 @@
 <?xml version="1.0"?>
 <robot xmlns:xacro="http://www.ros.org/wiki/xacro" >
-    <xacro:property name="tilt_deg_cam" value="25"/>
+    <xacro:property name="tilt_deg_cam" value="20"/>
     <xacro:property name="tilt_rad_cam" value="${tilt_deg_cam * pi / 180.0}"/>
     <joint name="camera_joint" type="fixed">

Commit message: update camera urdf

File: src/robocops_description/description/urdf/camera.xacro (robot description, xacro)
@@ -1,5 +1,5 @@
 <?xml version="1.0"?>
 <robot xmlns:xacro="http://www.ros.org/wiki/xacro" >
-    <xacro:property name="tilt_deg_cam" value="20"/>
+    <xacro:property name="tilt_deg_cam" value="22"/>
     <xacro:property name="tilt_rad_cam" value="${tilt_deg_cam * pi / 180.0}"/>
     <joint name="camera_joint" type="fixed">

Commit message: fix camera tilt

File: src/robocops_description/description/urdf/camera.xacro (robot description, xacro)
@@ -1,5 +1,5 @@
 <?xml version="1.0"?>
 <robot xmlns:xacro="http://www.ros.org/wiki/xacro" >
-    <xacro:property name="tilt_deg_cam" value="22"/>
+    <xacro:property name="tilt_deg_cam" value="21"/>
     <xacro:property name="tilt_rad_cam" value="${tilt_deg_cam * pi / 180.0}"/>
     <joint name="camera_joint" type="fixed">

Commit message: some params

File: src/robocops_description/description/urdf/camera.xacro (robot description, xacro)
@@ -1,5 +1,5 @@
 <?xml version="1.0"?>
 <robot xmlns:xacro="http://www.ros.org/wiki/xacro" >
-    <xacro:property name="tilt_deg_cam" value="21"/>
+    <xacro:property name="tilt_deg_cam" value="22"/>
     <xacro:property name="tilt_rad_cam" value="${tilt_deg_cam * pi / 180.0}"/>
     <joint name="camera_joint" type="fixed">
